Commit message: modified:   description/lidar.xacro 	modified:   description/robot_core.xacro

File: description/lidar.xacro (robot description, xacro)
@@ -1,19 +1,17 @@
 <?xml version="1.0"?>
-<robot xmlns:xacro="http://www.ros.org/wiki/xacro"  name="robot">
+<robot xmlns:xacro="http://www.ros.org/wiki/xacro" >
     <joint name="laser_joint" type="fixed">
+        <parent link="chassis"/>
+        <child link="laser_frame"/>
         <origin xyz="0.1 0 0.175" rpy="0 0 0"/>
-        <parent link="chassis"/>
-        <child link="laser"/>
     </joint>
-    <link name="laser">
+    <link name="laser_frame">
         <visual>
-            <origin xyz="0 0 0" rpy="0 0 0"/>
             <geometry>
                 <cylinder radius="0.05" length="0.04"/>
             </geometry>
-            <material name="black"/>
+            <material name="red"/>
         </visual>
         <collision>
-            <origin xyz="0 0 0" rpy="0 0 0"/>
             <geometry>
                 <cylinder radius="0.05" length="0.04"/>
@@ -24,6 +22,6 @@
         </xacro:inertial_cylinder>
     </link>
-    <gazebo reference="laser">
-        <material>Gazebo/Black</material>
+    <gazebo reference="laser_frame">
+        <material>Gazebo/Red</material>
         <sensor name="laser" type="ray">
             <pose> 0 0 0 0 0 0 </pose>

File: description/robot_core.xacro (robot description, xacro)
@@ -13,4 +13,7 @@
     <material name="black">
         <color rgba="0 0 0 1"/>
+    </material>
+    <material name="red">
+        <color rgba="1 0 0 0"/>
     </material>
     <!-- BASE LINK -->
